File: project/LoRa-GPS-Tracker.kicad_sch (KiCad schematic)
At the start: 53 parts, among them IC1 MCP73831-2-OT, IC103 FT230XS, IC104 NCP705MT30TCG, IC2 MCP100-300D, M1 SIM28ML, M102 RAK3172, Q101 BSS123, Q102 TP0610K, Q103 BSH205G2VL, SW101 ON / OFF, X1 USB_B_Micro, X103 +, X104 -, X3 Conn_Coaxial, X3 DEBUG

Commit message: Hardware: - Add RESET line for SWD interface - Replace micro USB with USB C
Software:
- Add firmware for LoRa-GPS-Tracker PCB

Signed-off-by: Daniel Kampert <DanielKampert@kampis-elektroecke.de>
Parts:
- removed X1: USB_B_Micro, Wuerth:629105150521, symbol Connector:USB_B_Micro
- added AE102: LoRa Antenna (434 MHz), symbol Device:Antenna
- added R107, R108: 5k1, Resistor_SMD:R_0603_1608Metric, symbol Device:R_Small
- added X101: DEBUG, Connector_USB:USB_C_Receptacle_GCT_USB4105-xx-A_16P_TopMnt_Horizontal, symbol Connector:USB_C_Receptacle_USB2.0
- JP101: value ~ -> RX
- JP102: value ~ -> TX
- JP103: value PROG -> BOOT
- M102: Distributor (none) -> RAK Wireless; Order Number (none) -> 301025
- R101: renamed from R103; now not fitted
- R111: renamed from R107; value 2k -> 10k; Mfr. No. RC0402JR-072KL -> RC0402JR-0710KL; Order Number 603-RC0402JR-072KL -> 603-RC0402JR-0710KL
- renumbered C105 to C104, C104 to C105, C109 to C108, C108 to C109, R101 to R102, R102 to R103, R108 to R109, R109 to R110, R110 to R112, R111 to R113, R112 to R114, R113 to R115, R114 to R116, R115 to R117, R116 to R118, R117 to R119
Connections:
- net +3V0: no longer IC103.11 (~{RESET})
- net GND: now also R107.2, R108.1, X101.A1 (GND), X101.A12 (GND), X101.B1 (GND), X101.B12 (GND), X101.S1 (SHIELD); no longer D101.1 (K)
- net USB_DM: now also X101.A7 (D-), X101.B7 (D-)
- net USB_DP: now also X101.A6 (D+), X101.B6 (D+)
- net V_USB: now also D101.2 (A), X101.A4 (VBUS), X101.A9 (VBUS), X101.B4 (VBUS), X101.B9 (VBUS)
- net at SW101.1: now also IC104.4 (EN), R115.1; no longer R115.2
- net at C108.1, IC103.10 (3V3OUT): now also IC103.11 (~{RESET})
- net at R112.2: now also D101.1 (K); no longer D101.2 (A)
- net ~{RESET}: now reaches X3.10 (~{RESET})
- net ~{RESET}: now also C113.1, M102.22 (~{RST}), R118.2
- new net: IC2.1 (~{RST}), R115.2
- new net: R108.2, X101.B5 (CC2)
- new net: R107.1, X101.A5 (CC1)
- no-connect marks 32 -> 33
Other:
- note added: "NOTE: Charge current is limited to 100 mA."
- moved on the sheet: AE101, C101, C105, C108, C109, C111, C112, D101, IC1, IC104, IC2, Q103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
